File: KiCadTrial.kicad_pcb (KiCad board)
At the start: 2 copper layers, 13 x 16 mm, 3 parts, among them J1 Conn_01x02

Commit message: Conn V2
numbered the pins of the connector on the bottom silkscreen layer
Parts:
- J1: footprint Connector_Molex:Molex_KK-254_AE-6410-02A_1x02_P2.54mm_Vertical -> myPCBLib:Molex_KK-254_AE-6410-02A_1x02_P2.54mm_Vertical
- R1: value R_Photo -> 330
Connections:
- D1 pad C: Net-(D1-Cathode) -> unconnected-(D1-Cathode-PadC)
- R1 pad 1: Net-(D1-Cathode) -> unconnected-(R1-Pad1)
Changed lines of the file:
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@@
   (net 1 "GND")
   (net 2 "+3.3V")
-  (net 3 "Net-(D1-Cathode)")
+  (net 3 "unconnected-(D1-Cathode-PadC)")
+  (net 4 "unconnected-(R1-Pad1)")
   (footprint "myPCBLib:LED0603" (layer "F.Cu")
     (at 160 110.175 90)
     (descr "Surface Mount LED 0603 - white")
     (tags "optical electronics")
+    (property "JLCPCB" "C965805")
+    (property "MPN" "XL-1608SYGC-06")
+    (property "Manufacturer" "XINGLIGHT")
     (property "PN" "EKT_426738")
     (property "Sheetfile" "KiCadTrial.kicad_sch")
@@
       (net 1 "GND") (pinfunction "Anode") (pintype "passive") (thermal_bridge_angle 45))
     (pad "C" smd rect (at -0.825 0 90) (size 0.8 0.8) (layers "F.Cu" "F.Paste" "F.Mask")
-      (net 3 "Net-(D1-Cathode)") (pinfunction "Cathode") (pintype "passive") (thermal_bridge_angle 45))
+      (net 3 "unconnected-(D1-Cathode-PadC)") (pinfunction "Cathode") (pintype "passive") (thermal_bridge_angle 45))
     (model "${KICAD6_3DMODEL_DIR}/LED_SMD.3dshapes/LED_0603_1608Metric.wrl"
       (offset (xyz 0 0 0))
@@
     )
   )
-  (footprint "Connector_Molex:Molex_KK-254_AE-6410-02A_1x02_P2.54mm_Vertical" (layer "F.Cu")
+  (footprint "myPCBLib:Molex_KK-254_AE-6410-02A_1x02_P2.54mm_Vertical" (layer "F.Cu")
     (at 156.46 104)
     (descr "Molex KK-254 Interconnect System, old/engineering part number: AE-6410-02A example for new part number: 22-27-2021, 2 Pins (http://www.molex.com/pdm_docs/sd/022272021_sd.pdf), generated with kicad-footprint-generator")
     (tags "connector Molex KK-254 vertical")
+    (property "JLCPCB" "C5116481")
+    (property "MPN" "2.54-1*2")
+    (property "Manufacturer" "ZHOURI")
+    (property "PN" "anything")
     (property "Sheetfile" "KiCadTrial.kicad_sch")
     (property "Sheetname" "")
@@
     (fp_text value "Conn_01x02" (at 1.27 4.08) (layer "F.Fab")
         (effects (font (size 1 1) (thickness 0.15)))
+    )
+    (fp_text user "2" (at 3.09 -1.04 unlocked) (layer "B.SilkS")
+        (effects (font (size 1 1) (thickness 0.1)) (justify left bottom mirror))
+    )
+    (fp_text user "1" (at 0.48 -1.04 unlocked) (layer "B.SilkS")
+        (effects (font (size 1 1) (thickness 0.1)) (justify left bottom mirror))
     )
     (fp_text user "${REFERENCE}" (at 1.27 -2.22) (layer "F.Fab")
@@
     (descr "Resistor SMD 0805 (2012 Metric), square (rectangular) end terminal, IPC_7351 nominal, (Body size source: IPC-SM-782 page 72, https://www.pcb-3d.com/wordpress/wp-content/uploads/ipc-sm-782a_amendment_1_and_2.pdf), generated with kicad-footprint-generator")
     (tags "resistor")
+    (property "JLCPCB" "C23138")
+    (property "MPN" "0603WAF3300T5E")
+    (property "Manufacturer" "UNI-ROYAL(Uniroyal Elec)")
+    (property "PN" "something")
     (property "Sheetfile" "KiCadTrial.kicad_sch")
     (property "Sheetname" "")
@@
         (effects (font (size 1 1) (thickness 0.15)))
     )
-    (fp_text value "R_Photo" (at 0 1.65 90) (layer "F.Fab")
+    (fp_text value "330" (at 0 1.65 90) (layer "F.Fab")
         (effects (font (size 1 1) (thickness 0.15)))
     )
@@
       (stroke (width 0.1) (type solid)) (layer "F.Fab"))
     (pad "1" smd roundrect (at -0.9125 0 90) (size 1.025 1.4) (layers "F.Cu" "F.Paste" "F.Mask") (roundrect_rratio 0.243902439)
-      (net 3 "Net-(D1-Cathode)") (pintype "passive"))
+      (net 4 "unconnected-(R1-Pad1)") (pintype "passive"))
     (pad "2" smd roundrect (at 0.9125 0 90) (size 1.025 1.4) (layers "F.Cu" "F.Paste" "F.Mask") (roundrect_rratio 0.243902439)
       (net 2 "+3.3V") (pintype "passive"))

Commit message: Led polarity correction
changed the polarity of the led connected between the resistor and the gnd
Connections:
- D1 pad A: GND -> Net-(D1-Anode)
- D1 pad C: unconnected-(D1-Cathode-PadC) -> GND
- R1 pad 1: unconnected-(R1-Pad1) -> Net-(D1-Anode)
Changed lines of the file:
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@@
   (net 1 "GND")
   (net 2 "+3.3V")
-  (net 3 "unconnected-(D1-Cathode-PadC)")
-  (net 4 "unconnected-(R1-Pad1)")
+  (net 3 "Net-(D1-Anode)")
   (footprint "myPCBLib:LED0603" (layer "F.Cu")
     (at 160 110.175 90)
@@
       (stroke (width 0.1) (type solid)) (fill solid) (layer "F.CrtYd"))
     (pad "A" smd rect (at 0.825 0 90) (size 0.8 0.8) (layers "F.Cu" "F.Paste" "F.Mask")
-      (net 1 "GND") (pinfunction "Anode") (pintype "passive") (thermal_bridge_angle 45))
+      (net 3 "Net-(D1-Anode)") (pinfunction "Anode") (pintype "passive") (thermal_bridge_angle 45))
     (pad "C" smd rect (at -0.825 0 90) (size 0.8 0.8) (layers "F.Cu" "F.Paste" "F.Mask")
-      (net 3 "unconnected-(D1-Cathode-PadC)") (pinfunction "Cathode") (pintype "passive") (thermal_bridge_angle 45))
+      (net 1 "GND") (pinfunction "Cathode") (pintype "passive") (thermal_bridge_angle 45))
     (model "${KICAD6_3DMODEL_DIR}/LED_SMD.3dshapes/LED_0603_1608Metric.wrl"
       (offset (xyz 0 0 0))
@@
       (stroke (width 0.1) (type solid)) (layer "F.Fab"))
     (pad "1" smd roundrect (at -0.9125 0 90) (size 1.025 1.4) (layers "F.Cu" "F.Paste" "F.Mask") (roundrect_rratio 0.243902439)
-      (net 4 "unconnected-(R1-Pad1)") (pintype "passive"))
+      (net 3 "Net-(D1-Anode)") (pintype "passive"))
     (pad "2" smd roundrect (at 0.9125 0 90) (size 1.025 1.4) (layers "F.Cu" "F.Paste" "F.Mask") (roundrect_rratio 0.243902439)
       (net 2 "+3.3V") (pintype "passive"))
